File: electronics/isimud_main/isimud_main.kicad_pcb (KiCad board)
At the start: 2 copper layers, 160.3 x 110.1 mm, 95 parts, among them CON1 12V DC, IC1 ENC28J60-I/SO, J1 DB9, J2 RJ45-TRANSFO, J3 DB9, P1 CONN_02X50, P2 LIPO_BAT, P3 SAT MODULE GPS, P4 UART_0, P5 UART_4, P6 ETH_CLKOUT, P7 RS232-UART, P8 RS232-2, P9 AKTIF GPS ANTEN, U1 SOM-A20, U2 SIMCARD_HOLDER, U3 MAX232, U4 LM2576, U5 LM2576, X1 CRYSTAL_SMD

Commit message: pcb rev.a produced,mechanics design has began
Routing:
- net Net-(C2-Pad1): track 41.2 -> 26.8 mm, vias 3 -> 1
Other:
- net class Default: clearance 0.2 -> 0.01
- net class POWER: clearance 0.2 -> 0.01
- rule trace_clearance: 0.2 -> 0.01
- rule via_min_drill: 0.6 -> 0.3
- rule via_min_size: 1.2 -> 0.3
Changed lines of the file:
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@@
     (links 255)
     (no_connects 0)
-    (area 48.514 20.806999 235.966001 152.501601)
+    (area 48.514 20.996999 235.966001 152.501601)
     (thickness 1.6)
     (drawings 17)
-    (tracks 1306)
+    (tracks 1298)
     (zones 0)
     (modules 95)
@@
     (33 F.Adhes user)
     (34 B.Paste user)
-    (35 F.Paste user)
+    (35 F.Paste user hide)
     (36 B.SilkS user)
     (37 F.SilkS user)
@@
   (setup
     (last_trace_width 0.4)
-    (trace_clearance 0.2)
+    (trace_clearance 0.01)
     (zone_clearance 0.7)
     (zone_45_only yes)
@@
     (via_size 1.2)
     (via_drill 0.8)
-    (via_min_size 1.2)
-    (via_min_drill 0.6)
+    (via_min_size 0.3)
+    (via_min_drill 0.3)
+    (blind_buried_vias_allowed yes)
     (uvia_size 0.3)
     (uvia_drill 0.1)
@@
     (visible_elements FFFFFF7F)
     (pcbplotparams
-      (layerselection 0x00030_80000001)
+      (layerselection 0x3ffff_80000001)
       (usegerberextensions false)
       (excludeedgelayer true)
       (linewidth 0.100000)
       (plotframeref false)
-      (viasonmask false)
+      (viasonmask true)
       (mode 1)
       (useauxorigin false)
@@
       (plotvalue true)
       (plotinvisibletext false)
-      (padsonsilk false)
+      (padsonsilk true)
       (subtractmaskfromsilk false)
-      (outputformat 4)
+      (outputformat 1)
       (mirror false)
       (drillshape 0)
       (scaleselection 1)
-      (outputdirectory output/pdf/))
+      (outputdirectory output))
   )
   (net 0 "")
@@
   (net 356 "Net-(C13-Pad2)")
   (net_class Default "This is the default net class."
-    (clearance 0.2)
+    (clearance 0.01)
     (trace_width 0.4)
     (via_dia 1.2)
@@
   )
   (net_class POWER ""
-    (clearance 0.2)
+    (clearance 0.01)
     (trace_width 0.5)
     (via_dia 1.2)
@@
   (segment (start 123.1693 130.4417) (end 123.8043 130.4417) (width 0.5) (layer B.Cu) (net 3))
   (via (at 127.198 89.7752) (size 1.2) (layers F.Cu B.Cu) (net 4))
-  (via (at 116.733 64.9875) (size 1.2) (layers F.Cu B.Cu) (net 4))
+  (via (at 116.733 64.9875) (size 1.2) (drill 0.8) (layers F.Cu B.Cu) (net 4))
   (segment (start 126.916 75.1706) (end 116.733 64.9875) (width 0.5) (layer B.Cu) (net 4))
   (segment (start 126.916 89.4931) (end 126.916 75.1706) (width 0.5) (layer B.Cu) (net 4))
@@
   (segment (start 99.7382 67.7211) (end 115.209 83.1922) (width 0.5) (layer F.Cu) (net 4))
   (segment (start 99.7382 66.421) (end 99.7382 67.7211) (width 0.5) (layer F.Cu) (net 4))
-  (via (at 101.216 64.7909) (size 1.2) (layers F.Cu B.Cu) (net 5))
-  (via (at 98.6915 48.2497) (size 1.2) (layers F.Cu B.Cu) (net 5))
+  (via (at 101.216 64.7909) (size 1.2) (drill 0.8) (layers F.Cu B.Cu) (net 5))
+  (via (at 98.6915 48.2497) (size 1.2) (drill 0.8) (layers F.Cu B.Cu) (net 5))
   (segment (start 114.769 48.2497) (end 98.6915 48.2497) (width 0.4) (layer F.Cu) (net 5))
   (segment (start 115.019 48.5001) (end 114.769 48.2497) (width 0.4) (layer F.Cu) (net 5))
@@
   (segment (start 140.491 94.6374) (end 141.866 96.012) (width 0.5) (layer F.Cu) (net 27))
   (segment (start 140.491 94.5521) (end 140.491 94.6374) (width 0.5) (layer F.Cu) (net 27))
-  (via (at 128.949 72.4748) (size 1.2) (layers F.Cu B.Cu) (net 28))
+  (via (at 128.949 72.4748) (size 1.2) (drill 0.8) (layers F.Cu B.Cu) (net 28))
   (segment (start 209.551 59.182) (end 211.051 59.182) (width 0.5) (layer F.Cu) (net 28))
   (segment (start 211.051 59.182) (end 211.051 54.3112) (width 0.5) (layer F.Cu) (net 28))
@@
   (segment (start 195.834 132.842) (end 192.024 132.842) (width 0.5) (layer F.Cu) (net 149))
   (segment (start 199.009 136.017) (end 195.834 132.842) (width 0.5) (layer F.Cu) (net 149))
-  (via (at 89.0997 44.0337) (size 1.2) (layers F.Cu B.Cu) (net 283))
+  (via (at 89.0997 44.0337) (size 1.2) (drill 0.8) (layers F.Cu B.Cu) (net 283))
   (via (at 144.63522 131.12496) (size 1.2) (layers F.Cu B.Cu) (net 283))
   (segment (start 143.893 131.572) (end 142.494 131.572) (width 0.5) (layer F.Cu) (net 283))
@@
   (segment (start 144.63522 129.58318) (end 143.66494 129.58318) (width 0.4) (layer B.Cu) (net 285))
   (segment (start 143.66494 129.58318) (end 141.638 127.55624) (width 0.4) (layer B.Cu) (net 285))
-  (via (at 108.929 50.9694) (size 1.2) (layers F.Cu B.Cu) (net 285))
+  (via (at 108.929 50.9694) (size 1.2) (drill 0.8) (layers F.Cu B.Cu) (net 285))
   (via (at 144.63522 129.58318) (size 1.2) (layers F.Cu B.Cu) (net 285))
   (segment (start 129.999 72.0396) (end 108.929 50.9694) (width 0.5) (layer B.Cu) (net 285))
@@
   (segment (start 88.599 41.529) (end 88.599 42.679) (width 0.5) (layer F.Cu) (net 285))
   (via (at 160.528 56.8536) (size 1.2) (layers F.Cu B.Cu) (net 347))
-  (via (at 81.6905 55.9572) (size 1.2) (layers F.Cu B.Cu) (net 347))
+  (via (at 81.6905 55.9572) (size 1.2) (drill 0.8) (layers F.Cu B.Cu) (net 347))
   (via (at 195.934 108.441) (size 1.2) (layers F.Cu B.Cu) (net 347))
   (segment (start 66.2804 48.848) (end 65.024 48.848) (width 0.5) (layer F.Cu) (net 347))
@@
   (via (at 115.1001 124.0917) (size 1.2) (drill 0.8) (layers F.Cu B.Cu) (net 350))
   (segment (start 120.8638 118.328) (end 115.1001 124.0917) (width 0.3) (layer F.Cu) (net 350))
-  (via (at 129.997 126.289) (size 1.2) (layers F.Cu B.Cu) (net 350))
-  (segment (start 129.997 128.067) (end 129.997 126.289) (width 0.4) (layer F.Cu) (net 350))
-  (segment (start 126.594 130.404) (end 129.997 128.067) (width 0.4) (layer F.Cu) (net 350))
-  (segment (start 129.997 126.289) (end 129.235 125.527) (width 0.4) (layer B.Cu) (net 350))
-  (segment (start 129.235 125.527) (end 129.235 122.326) (width 0.4) (layer B.Cu) (net 350))
-  (via (at 129.235 122.326) (size 1.2) (layers F.Cu B.Cu) (net 350))
-  (segment (start 129.946 121.615) (end 129.946 118.364) (width 0.4) (layer F.Cu) (net 350))
-  (segment (start 129.235 122.326) (end 129.946 121.615) (width 0.4) (layer F.Cu) (net 350))
   (segment (start 127.694 118.364) (end 129.946 118.364) (width 0.5) (layer F.Cu) (net 350))
   (segment (start 127.658 118.328) (end 127.694 118.364) (width 0.5) (layer F.Cu) (net 350))

Commit message: test 0.1
Other:
- board text added: "TX2 RX2 TX1 RX1"
- board text removed: "TX1 RX1 TX2 RX2"
Changed lines of the file:
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@@
     (tags "Tantal Cap. , Size D, EIA-7343, Hand Soldering,")
     (attr smd)
-    (fp_text reference C3 (at -0.20066 -3.29946 180) (layer F.SilkS)
+    (fp_text reference C3 (at -0.2667 3.4544 180) (layer F.SilkS)
       (effects (font (size 1 1) (thickness 0.15)))
     )
@@
     (descr "SMT capacitor, aluminium electrolytic, 6.3x5.8")
     (attr smd)
-    (fp_text reference C4 (at 5.9944 -0.2538 270) (layer F.SilkS)
+    (fp_text reference C4 (at 6.3119 -2.5144 270) (layer F.SilkS)
       (effects (font (size 1 1) (thickness 0.15)))
     )
@@
     (descr "SMT capacitor, aluminium electrolytic, 6.3x5.8")
     (attr smd)
-    (fp_text reference C11 (at 0 -4.445 270) (layer F.SilkS)
+    (fp_text reference C11 (at -0.4064 -5.4229 270) (layer F.SilkS)
       (effects (font (size 1 1) (thickness 0.15)))
     )
@@
       (effects (font (size 1 1) (thickness 0.15)))
     )
-    (fp_text value "SAT MODULE GPS" (at 0 8.89) (layer F.Fab)
+    (fp_text value "SAT MODULE GPS" (at -0.1524 8.306) (layer F.Fab)
       (effects (font (size 1 1) (thickness 0.15)))
     )
@@
     (effects (font (size 1.5 1.5) (thickness 0.3)))
   )
-  (gr_text "TX1\nRX1\nTX2\nRX2" (at 95.4024 56.1848) (layer F.SilkS)
+  (gr_text "TX2\nRX2\nTX1\nRX1" (at 95.4024 56.1848) (layer F.SilkS)
     (effects (font (size 1.5 1.5) (thickness 0.3)))
   )
