File: electronics/isimud_main/isimud_main.kicad_pcb (KiCad board)
At the start: 2 copper layers, 160.3 x 110.1 mm, 95 parts, among them CON1 12V DC, IC1 ENC28J60-I/SO, J1 DB9, J2 RJ45-TRANSFO, J3 DB9, P1 CONN_02X50, P2 LIPO_BAT, P3 SAT MODULE GPS, P4 UART_0, P5 UART_4, P6 ETH_CLKOUT, P7 RS232-UART, P8 RS232-2, P9 AKTIF GPS ANTEN, U1 SOM-A20, U2 SIMCARD_HOLDER, U3 MAX232, U4 LM2576, U5 LM2576, X1 CRYSTAL_SMD

Commit message: shematics is done,pcb routing started
Parts:
- removed C30, C36, C39: 100nF, Capacitors_SMD:C_0805_HandSoldering
- removed C31, C32: 18pF, Capacitors_SMD:C_0805_HandSoldering
- removed IC1: ENC28J60-I/SO, Housings_SOIC:SOIC-28_7.5x17.9mm_Pitch1.27mm
- removed L4: 100uH, Inductors:SELF-WE-PD-XXL
- removed L6: ferrite bead, Air_Coils_SML_NEOSID:Neosid_Air-Coil_SML_2turn_HAM0231A
- removed P6: ETH_CLKOUT, Pin_Headers:Pin_Header_Straight_1x01
- removed R12: 1k, Resistors_SMD:R_0805_HandSoldering
- removed R22: 100k, Resistors_SMD:R_0805_HandSoldering
- removed R23: 10k, Resistors_SMD:R_0805_HandSoldering
- removed R24: 2k2 %1, Resistors_SMD:R_0805_HandSoldering
- removed R25, R26, R27, R29: 49.9 %1, Resistors_SMD:R_0805_HandSoldering
- removed R28, R30: 180R, Resistors_SMD:R_0805_HandSoldering
- removed R31: 0R, Resistors_SMD:R_0805_HandSoldering
- removed X1: CRYSTAL_SMD, Crystals:Crystal_HC52-U_Vertical
- added C15: 100uF, Capacitors_SMD:c_elec_6.3x5.8, F.Cu at (119.1, 74.3)
- added C24: 1000uF 16V, Capacitors_ThroughHole:C_Radial_D10_L16_P5, F.Cu at (89.3, 48.3)
- added C25: 220uF 16V, Capacitors_SMD:c_elec_6.3x5.8, F.Cu at (110.5, 83.7)
- added C41, C43, C50, C51, C54, C55, C56, C57, C58, C59: 100nF, Capacitors_SMD:C_0603_HandSoldering, F.Cu at (136.5, 153.5)
- added C42, C65: NA, Capacitors_SMD:C_0603_HandSoldering, F.Cu at (136.5, 153.5)
- added C48, C53: 22uF/6.3V, Capacitors_SMD:C_0603_HandSoldering, F.Cu at (136.5, 153.5)
- added C52: 22uF/6.3V, Capacitors_SMD:C_0603_HandSoldering, F.Cu at (227.7, 104.3)
- added C61: 100nF, Capacitors_SMD:C_0603_HandSoldering, B.Cu at (227.6, 50.7)
- added C62, C64: 27pF, Capacitors_SMD:C_0603_HandSoldering, F.Cu at (136.5, 153.5)
- added C71: 1nF/2kV/X7R/1206, Capacitors_SMD:C_1206_HandSoldering, F.Cu at (203.0, 62.3)
- added D7: 1N5822, Diodes_SMD:SMB_Handsoldering, F.Cu at (94.8, 70.2)
- added L11: FB0805/600R/2A, Capacitors_SMD:C_0805_HandSoldering, F.Cu at (225.1, 89.6)
- added L12, L13: FB0805/600R/2A, Capacitors_SMD:C_0805_HandSoldering, F.Cu at (136.5, 153.5)
- added L14: 4.7uH/1.15A/DCR<0.1R/CD43, Inductors:Inductor_1212, F.Cu at (234.3, 74.8)
- added Q1: E4SB25.000F20E15(25MHz/20pF/20ppm/5x3.2mm), Capacitors_SMD:C_2220_HandSoldering, F.Cu at (234.1, 80.0)
- added R40: 10K, Resistors_SMD:R_0603_HandSoldering, F.Cu at (136.5, 153.5)
- added R41, R42, R66: 22R, Resistors_SMD:R_0603_HandSoldering, F.Cu at (136.5, 153.5)
- added R43: 10k, Resistors_SMD:R_0603_HandSoldering, F.Cu at (136.5, 153.5)
- added R44, R57, R60, R64: NA, Resistors_SMD:R_0603_HandSoldering, F.Cu at (136.5, 153.5)
- added R47, R49, R61: 1K, Resistors_SMD:R_0603_HandSoldering, F.Cu at (136.5, 153.5)
- added R48, R59, R62: 4K7, Resistors_SMD:R_0603_HandSoldering, F.Cu at (136.5, 153.5)
- added R52: 2.49k/1%, Resistors_SMD:R_0603_HandSoldering, F.Cu at (136.5, 153.5)
- added R63: 1k, Resistors_SMD:R_0603_HandSoldering, F.Cu at (136.5, 153.5)
- added R65: NA(4.7k), Resistors_SMD:R_0603_HandSoldering, F.Cu at (136.5, 153.5)
- added RM4G1, RM4G2, RM4G3: R, Resistors_SMD:R_0603_HandSoldering, F.Cu at (136.5, 153.5)
- added RM5G1, RM5G2, RM5G3, RM5G4: RA1206_(4X0603)_4B8_22R, Resistors_SMD:R_0603_HandSoldering, F.Cu at (136.5, 153.5)
- added U7: RTL8211CL-GR, Housings_QFP:LQFP-48_7x7mm_Pitch0.5mm, F.Cu at (234.9, 91.8)
- added U8: LM2576-5V, TO_SOT_Packages_THT:Pentawatt_Neutral_Straight_Vertical_TO220-5-T05A, F.Cu at (107.8, 73.4)
- C20: footprint Capacitors_ThroughHole:C_Radial_D10_L13_P5 -> Capacitors_ThroughHole:C_Radial_D10_L16_P5
- C22: footprint Capacitors_Tantalum_SMD:TantalC_SizeB_EIA-3528_HandSoldering -> Capacitors_ThroughHole:C_Radial_D10_L16_P5
- C33: value 100nF -> 22uF/6.3V; footprint Capacitors_SMD:C_0805_HandSoldering -> Capacitors_SMD:C_0603_HandSoldering
- C34, C35: footprint Capacitors_SMD:C_0805_HandSoldering -> Capacitors_SMD:C_0603_HandSoldering
- C37: value 10uF -> 22uF/6.3V; footprint Capacitors_Tantalum_SMD:TantalC_SizeD_EIA-7343_HandSoldering -> Capacitors_SMD:C_0603_HandSoldering
- C38: value 10nF -> 100nF; footprint Capacitors_SMD:C_0805_HandSoldering -> Capacitors_SMD:C_0603_HandSoldering
- J2: value RJ45-TRANSFO -> TM211Q01FM22; footprint KiCAD connector library:RJHSE538X -> rj45:TM211Q01FM22
- R10: value 2k -> NA
- R11: value 1k -> 0R
- U4: value LM2576 -> LM2576-5V
- moved J2 51.8 mm to (233.1, 44.7)
- moved C22 14.4 mm to (82.1, 81.7)
- moved D2 1.45 mm to (89.7, 70.1)
Connections:
- net Net-(R10-Pad1) renamed ETXCK
- C20 pad 1: Net-(C20-Pad1) -> PWR_LED
- C22 pad 1: Net-(C22-Pad1) -> +6V
- C33 pad 1: +3V3 -> GND
- C33 pad 2: GND -> Net-(C33-Pad2)
- C34 pad 1: +3V3 -> GND
- C34 pad 2: GND -> Net-(C33-Pad2)
- C35 pad 1: +3V3 -> GND
- C35 pad 2: GND -> Net-(C33-Pad2)
- C37 pad 1: Net-(C37-Pad1) -> GND
- C37 pad 2: GND -> Net-(C37-Pad2)
- C38 pad 1: Net-(C38-Pad1) -> GND
- C38 pad 2: GND -> Net-(C37-Pad2)
- J1 pad 1: Net-(J1-Pad1) -> (no net)
- J1 pad 4: Net-(J1-Pad4) -> (no net)
- J1 pad 6: Net-(J1-Pad6) -> (no net)
- J1 pad 7: Net-(J1-Pad7) -> (no net)
- J1 pad 8: Net-(J1-Pad8) -> (no net)
- J1 pad 9: Net-(J1-Pad9) -> (no net)
- J2 pad 1: ETH_TPOUT+ -> Net-(J2-Pad1)
- J2 pad 13: GND -> Net-(J2-Pad13)
- J2 pad 3: ETH_TPOUT- -> Net-(J2-Pad3)
- J2 pad 4: ETH_TPIN+ -> Net-(J2-Pad4)
- J2 pad 6: ETH_TPIN- -> Net-(C61-Pad1)
- J2 pad 7: (no net) -> Net-(J2-Pad7)
- J3 pad 7: Net-(J3-Pad7) -> (no net)
- J3 pad 8: Net-(J3-Pad8) -> (no net)
- J3 pad 9: Net-(J3-Pad9) -> (no net)
- L1 pad 2: Net-(C20-Pad1) -> PWR_LED
- L2 pad 1: Net-(C20-Pad1) -> Net-(D7-Pad1)
- L2 pad 2: PWR_LED -> +5VD
- L3 pad 2: Net-(C22-Pad1) -> +6V
- P1 pad 1: Net-(P1-Pad1) -> (no net)
- P1 pad 10: Net-(P1-Pad10) -> (no net)
- P1 pad 11: Net-(P1-Pad11) -> (no net)
- P1 pad 12: Net-(P1-Pad12) -> (no net)
- P1 pad 13: Net-(P1-Pad13) -> (no net)
- P1 pad 14: Net-(P1-Pad14) -> (no net)
- P1 pad 15: Net-(P1-Pad15) -> (no net)
- P1 pad 16: Net-(P1-Pad16) -> (no net)
- P1 pad 17: Net-(P1-Pad17) -> (no net)
- P1 pad 18: Net-(P1-Pad18) -> (no net)
- P1 pad 19: Net-(P1-Pad19) -> (no net)
- P1 pad 2: Net-(P1-Pad2) -> (no net)
- P1 pad 20: Net-(P1-Pad20) -> (no net)
- P1 pad 21: Net-(P1-Pad21) -> (no net)
- P1 pad 23: Net-(P1-Pad23) -> (no net)
- P1 pad 25: Net-(P1-Pad25) -> (no net)
- P1 pad 26: Net-(P1-Pad26) -> (no net)
- P1 pad 27: Net-(P1-Pad27) -> (no net)
- P1 pad 29: Net-(P1-Pad29) -> (no net)
- P1 pad 3: Net-(P1-Pad3) -> (no net)
- P1 pad 30: Net-(P1-Pad30) -> (no net)
- P1 pad 31: Net-(P1-Pad31) -> (no net)
- P1 pad 32: Net-(P1-Pad32) -> (no net)
- P1 pad 33: Net-(P1-Pad33) -> (no net)
- P1 pad 34: Net-(P1-Pad34) -> (no net)
- P1 pad 36: Net-(P1-Pad36) -> (no net)
- P1 pad 37: Net-(P1-Pad37) -> (no net)
- P1 pad 38: Net-(P1-Pad38) -> (no net)
- P1 pad 39: Net-(P1-Pad39) -> (no net)
- P1 pad 4: Net-(P1-Pad4) -> (no net)
- P1 pad 40: Net-(P1-Pad40) -> (no net)
- P1 pad 41: Net-(P1-Pad41) -> (no net)
- P1 pad 42: Net-(P1-Pad42) -> (no net)
- P1 pad 43: Net-(P1-Pad43) -> (no net)
- P1 pad 44: Net-(P1-Pad44) -> (no net)
- P1 pad 45: Net-(P1-Pad45) -> (no net)
- P1 pad 46: Net-(P1-Pad46) -> (no net)
- P1 pad 47: Net-(P1-Pad47) -> (no net)
- P1 pad 48: Net-(P1-Pad48) -> (no net)
- P1 pad 49: Net-(P1-Pad49) -> (no net)
- P1 pad 5: Net-(P1-Pad5) -> (no net)
- P1 pad 52: Net-(P1-Pad52) -> (no net)
- P1 pad 53: Net-(P1-Pad53) -> (no net)
- P1 pad 54: Net-(P1-Pad54) -> (no net)
- P1 pad 55: Net-(P1-Pad55) -> (no net)
- P1 pad 56: Net-(P1-Pad56) -> (no net)
- P1 pad 6: Net-(P1-Pad6) -> (no net)
- P1 pad 61: Net-(P1-Pad61) -> (no net)
- P1 pad 63: Net-(P1-Pad63) -> (no net)
- P1 pad 66: Net-(P1-Pad66) -> (no net)
- P1 pad 7: Net-(P1-Pad7) -> (no net)
- P1 pad 71: Net-(P1-Pad71) -> (no net)
- P1 pad 72: Net-(P1-Pad72) -> (no net)
- P1 pad 74: Net-(P1-Pad74) -> (no net)
- P1 pad 78: Net-(P1-Pad78) -> (no net)
- P1 pad 8: Net-(P1-Pad8) -> (no net)
- P1 pad 80: Net-(P1-Pad80) -> (no net)
- P1 pad 84: Net-(P1-Pad84) -> (no net)
- P1 pad 9: Net-(P1-Pad9) -> (no net)
- P7 pad 1: Net-(P7-Pad1) -> UART3_TX
- P7 pad 2: Net-(P7-Pad2) -> UART3_RX
- P7 pad 3: UART3_RX -> Net-(P7-Pad3)
- P7 pad 4: UART3_TX -> Net-(P7-Pad4)
- R10 pad 2: Net-(C20-Pad1) -> Net-(R10-Pad2)
- R13 pad 2: Net-(C22-Pad1) -> +6V
- R5 pad 2: Net-(P7-Pad1) -> Net-(P7-Pad4)
- U1 pad 1-10: Net-(U1-Pad1-10) -> (no net)
- U1 pad 1-12: Net-(U1-Pad1-12) -> (no net)
- U1 pad 1-13: Net-(U1-Pad1-13) -> (no net)
- U1 pad 1-14: Net-(U1-Pad1-14) -> (no net)
- U1 pad 1-15: Net-(U1-Pad1-15) -> (no net)
- U1 pad 1-16: Net-(U1-Pad1-16) -> (no net)
- U1 pad 1-17: Net-(U1-Pad1-17) -> (no net)
- U1 pad 1-18: Net-(U1-Pad1-18) -> (no net)
- U1 pad 1-19: Net-(U1-Pad1-19) -> (no net)
- U1 pad 1-20: Net-(U1-Pad1-20) -> (no net)
- U1 pad 1-21: Net-(U1-Pad1-21) -> (no net)
- U1 pad 1-22: Net-(U1-Pad1-22) -> (no net)
- U1 pad 1-23: Net-(U1-Pad1-23) -> (no net)
- U1 pad 1-24: Net-(U1-Pad1-24) -> (no net)
- U1 pad 1-25: Net-(U1-Pad1-25) -> (no net)
- U1 pad 1-26: Net-(U1-Pad1-26) -> (no net)
- U1 pad 1-27: Net-(U1-Pad1-27) -> (no net)
- U1 pad 1-28: Net-(U1-Pad1-28) -> (no net)
- U1 pad 1-29: Net-(U1-Pad1-29) -> (no net)
- U1 pad 1-3: +3.3VADC -> (no net)
- U1 pad 1-30: Net-(U1-Pad1-30) -> (no net)
- U1 pad 1-31: Net-(U1-Pad1-31) -> (no net)
- U1 pad 1-32: Net-(U1-Pad1-32) -> (no net)
- U1 pad 1-33: Net-(U1-Pad1-33) -> (no net)
- U1 pad 1-34: Net-(U1-Pad1-34) -> (no net)
- U1 pad 1-35: Net-(U1-Pad1-35) -> (no net)
- U1 pad 1-36: Net-(U1-Pad1-36) -> (no net)
- U1 pad 1-37: Net-(U1-Pad1-37) -> (no net)
- U1 pad 1-38: Net-(U1-Pad1-38) -> (no net)
- U1 pad 1-39: Net-(U1-Pad1-39) -> (no net)
- U1 pad 1-40: Net-(U1-Pad1-40) -> (no net)
- U1 pad 1-6: Net-(U1-Pad1-6) -> (no net)
- U1 pad 1-7: Net-(U1-Pad1-7) -> (no net)
- U1 pad 1-8: Net-(U1-Pad1-8) -> (no net)
- U1 pad 2-10: Net-(U1-Pad2-10) -> (no net)
- U1 pad 2-11: Net-(U1-Pad2-11) -> (no net)
- U1 pad 2-12: Net-(U1-Pad2-12) -> (no net)
- U1 pad 2-13: Net-(U1-Pad2-13) -> (no net)
- U1 pad 2-14: Net-(U1-Pad2-14) -> (no net)
- U1 pad 2-15: Net-(U1-Pad2-15) -> (no net)
- U1 pad 2-16: Net-(U1-Pad2-16) -> (no net)
- U1 pad 2-17: Net-(U1-Pad2-17) -> (no net)
- U1 pad 2-18: Net-(U1-Pad2-18) -> (no net)
- U1 pad 2-19: Net-(U1-Pad2-19) -> (no net)
- U1 pad 2-20: Net-(U1-Pad2-20) -> (no net)
- U1 pad 2-23: SPI1_MISO -> ERXD0
- U1 pad 2-24: Net-(U1-Pad2-24) -> ETXD0
- U1 pad 2-25: SPI1_MOSI -> ERXD1
- U1 pad 2-26: Net-(U1-Pad2-26) -> ETXD1
- U1 pad 2-27: SPI1_CLK -> ERXD2
- U1 pad 2-28: Net-(U1-Pad2-28) -> ETXD2
- U1 pad 2-29: SPI1_CSO -> ERXD3
- U1 pad 2-30: Net-(U1-Pad2-30) -> ETXD3
- U1 pad 2-31: Net-(U1-Pad2-31) -> ERXDV
- U1 pad 2-32: Net-(U1-Pad2-32) -> ETXEN
- U1 pad 2-33: Net-(U1-Pad2-33) -> ERXCK
- U1 pad 2-34: Net-(U1-Pad2-34) -> Net-(R10-Pad2)
- U1 pad 2-35: Net-(U1-Pad2-35) -> (no net)
- U1 pad 2-36: Net-(U1-Pad2-36) -> Net-(R11-Pad2)
- U1 pad 2-37: Net-(U1-Pad2-37) -> (no net)
- U1 pad 2-38: Net-(U1-Pad2-38) -> CLK125
- U1 pad 2-39: Net-(U1-Pad2-39) -> (no net)
- U1 pad 2-40: Net-(U1-Pad2-40) -> EPHY-RST#
- U1 pad 2-5: Net-(U1-Pad2-5) -> (no net)
- U1 pad 2-6: Net-(U1-Pad2-6) -> (no net)
- U1 pad 2-7: Net-(U1-Pad2-7) -> (no net)
- U1 pad 2-8: Net-(U1-Pad2-8) -> (no net)
- U1 pad 2-9: Net-(U1-Pad2-9) -> (no net)
- U1 pad 3-10: Net-(U1-Pad3-10) -> (no net)
- U1 pad 3-11: Net-(U1-Pad3-11) -> (no net)
- U1 pad 3-12: Net-(U1-Pad3-12) -> (no net)
- U1 pad 3-13: Net-(U1-Pad3-13) -> (no net)
- U1 pad 3-14: Net-(U1-Pad3-14) -> (no net)
- U1 pad 3-15: Net-(U1-Pad3-15) -> (no net)
- U1 pad 3-16: Net-(U1-Pad3-16) -> (no net)
- U1 pad 3-17: Net-(U1-Pad3-17) -> (no net)
- U1 pad 3-18: Net-(U1-Pad3-18) -> (no net)
- U1 pad 3-19: Net-(U1-Pad3-19) -> (no net)
- U1 pad 3-2: Net-(U1-Pad3-2) -> (no net)
- U1 pad 3-20: Net-(U1-Pad3-20) -> (no net)
- U1 pad 3-21: Net-(U1-Pad3-21) -> (no net)
- U1 pad 3-22: Net-(U1-Pad3-22) -> (no net)
- U1 pad 3-23: Net-(U1-Pad3-23) -> (no net)
- U1 pad 3-24: Net-(U1-Pad3-24) -> (no net)
- U1 pad 3-25: Net-(U1-Pad3-25) -> (no net)
- U1 pad 3-26: Net-(U1-Pad3-26) -> (no net)
- U1 pad 3-27: Net-(U1-Pad3-27) -> (no net)
- U1 pad 3-28: Net-(U1-Pad3-28) -> (no net)
- U1 pad 3-29: Net-(U1-Pad3-29) -> (no net)
- U1 pad 3-30: Net-(U1-Pad3-30) -> (no net)
- U1 pad 3-31: Net-(U1-Pad3-31) -> (no net)
- U1 pad 3-32: Net-(U1-Pad3-32) -> (no net)
- U1 pad 3-33: Net-(U1-Pad3-33) -> (no net)
- U1 pad 3-34: Net-(U1-Pad3-34) -> (no net)
- U1 pad 3-35: Net-(U1-Pad3-35) -> (no net)
- U1 pad 3-36: Net-(U1-Pad3-36) -> (no net)
- U1 pad 3-37: Net-(U1-Pad3-37) -> (no net)
- U1 pad 3-38: Net-(U1-Pad3-38) -> (no net)
- U1 pad 3-39: Net-(U1-Pad3-39) -> (no net)
- U1 pad 3-4: Net-(U1-Pad3-4) -> (no net)
- U1 pad 3-40: Net-(U1-Pad3-40) -> (no net)
- U1 pad 3-6: Net-(U1-Pad3-6) -> (no net)
- U1 pad 3-7: Net-(U1-Pad3-7) -> STATUS_LED
- U1 pad 3-8: Net-(U1-Pad3-8) -> (no net)
- U1 pad 3-9: Net-(U1-Pad3-9) -> (no net)
- U1 pad 4-10: Net-(U1-Pad4-10) -> (no net)
- U1 pad 4-11: Net-(U1-Pad4-11) -> (no net)
- U1 pad 4-12: Net-(U1-Pad4-12) -> (no net)
- U1 pad 4-13: Net-(U1-Pad4-13) -> (no net)
- U1 pad 4-14: Net-(U1-Pad4-14) -> (no net)
- U1 pad 4-15: Net-(U1-Pad4-15) -> (no net)
- U1 pad 4-16: Net-(U1-Pad4-16) -> (no net)
- U1 pad 4-17: Net-(U1-Pad4-17) -> (no net)
- U1 pad 4-18: Net-(U1-Pad4-18) -> (no net)
- U1 pad 4-19: UART7_TX -> (no net)
- U1 pad 4-20: UART7_RX -> (no net)
- U1 pad 4-21: TWI1_SCK -> (no net)
- U1 pad 4-22: TWI1_SDA -> (no net)
- U1 pad 4-23: Net-(U1-Pad4-23) -> (no net)
- U1 pad 4-24: Net-(U1-Pad4-24) -> (no net)
- U1 pad 4-25: Net-(U1-Pad4-25) -> (no net)
- U1 pad 4-26: Net-(U1-Pad4-26) -> (no net)
- U1 pad 4-29: Net-(U1-Pad4-29) -> (no net)
- U1 pad 4-30: Net-(U1-Pad4-30) -> (no net)
- U1 pad 4-31: Net-(U1-Pad4-31) -> (no net)
- U1 pad 4-32: Net-(U1-Pad4-32) -> (no net)
- U1 pad 4-33: Net-(U1-Pad4-33) -> (no net)
- U1 pad 4-34: Net-(U1-Pad4-34) -> (no net)
- U1 pad 4-35: Net-(U1-Pad4-35) -> (no net)
- U1 pad 4-36: Net-(U1-Pad4-36) -> (no net)
- U1 pad 4-37: Net-(U1-Pad4-37) -> (no net)
- U1 pad 4-38: Net-(U1-Pad4-38) -> (no net)
- U1 pad 4-39: Net-(U1-Pad4-39) -> (no net)
- U1 pad 4-4: Net-(U1-Pad4-4) -> (no net)
- U1 pad 4-40: Net-(U1-Pad4-40) -> RESET_N
- U1 pad 4-5: Net-(U1-Pad4-5) -> (no net)
- U1 pad 4-6: Net-(U1-Pad4-6) -> (no net)
- U1 pad 4-7: Net-(U1-Pad4-7) -> (no net)
- U1 pad 4-8: Net-(U1-Pad4-8) -> (no net)
- U1 pad 4-9: Net-(U1-Pad4-9) -> (no net)
- U1 pad 5-10: Net-(U1-Pad5-10) -> (no net)
- U1 pad 5-11: PG5 -> (no net)
- U1 pad 5-12: Net-(U1-Pad5-12) -> (no net)
- U1 pad 5-14: Net-(U1-Pad5-14) -> (no net)
- U1 pad 5-16: Net-(U1-Pad5-16) -> (no net)
- U1 pad 5-18: Net-(U1-Pad5-18) -> (no net)
- U1 pad 5-20: Net-(U1-Pad5-20) -> (no net)
- U1 pad 5-22: Net-(U1-Pad5-22) -> (no net)
- U1 pad 5-24: Net-(U1-Pad5-24) -> (no net)
- U1 pad 5-25: Net-(U1-Pad5-25) -> (no net)
- U1 pad 5-26: Net-(U1-Pad5-26) -> (no net)
- U1 pad 5-27: Net-(U1-Pad5-27) -> (no net)
- U1 pad 5-28: Net-(U1-Pad5-28) -> (no net)
- U1 pad 5-29: Net-(U1-Pad5-29) -> (no net)
- U1 pad 5-30: Net-(U1-Pad5-30) -> (no net)
- U1 pad 5-31: Net-(U1-Pad5-31) -> (no net)
- U1 pad 5-32: Net-(U1-Pad5-32) -> (no net)
- U1 pad 5-33: Net-(U1-Pad5-33) -> (no net)
- U1 pad 5-34: Net-(U1-Pad5-34) -> (no net)
- U1 pad 5-35: Net-(U1-Pad5-35) -> (no net)
- U1 pad 5-36: Net-(U1-Pad5-36) -> (no net)
- U1 pad 5-37: Net-(U1-Pad5-37) -> (no net)
- U1 pad 5-38: Net-(U1-Pad5-38) -> (no net)
- U1 pad 5-39: Net-(U1-Pad5-39) -> (no net)
- U1 pad 5-4: Net-(U1-Pad5-4) -> (no net)
- U1 pad 5-40: Net-(U1-Pad5-40) -> (no net)
- U1 pad 5-6: Net-(U1-Pad5-6) -> (no net)
- U1 pad 5-8: Net-(U1-Pad5-8) -> (no net)
- U1 pad 6-10: Net-(U1-Pad6-10) -> (no net)
- U1 pad 6-11: Net-(U1-Pad6-11) -> (no net)
- U1 pad 6-12: Net-(U1-Pad6-12) -> (no net)
- U1 pad 6-13: Net-(U1-Pad6-13) -> (no net)
- U1 pad 6-14: Net-(U1-Pad6-14) -> (no net)
- U1 pad 6-15: Net-(U1-Pad6-15) -> (no net)
- U1 pad 6-16: Net-(U1-Pad6-16) -> (no net)
- U1 pad 6-17: Net-(U1-Pad6-17) -> (no net)
- U1 pad 6-18: Net-(U1-Pad6-18) -> (no net)
- U1 pad 6-19: Net-(U1-Pad6-19) -> (no net)
- U1 pad 6-20: Net-(U1-Pad6-20) -> (no net)
- U1 pad 6-21: Net-(U1-Pad6-21) -> (no net)
- U1 pad 6-22: Net-(U1-Pad6-22) -> (no net)
- U1 pad 6-23: Net-(U1-Pad6-23) -> (no net)
- U1 pad 6-24: Net-(U1-Pad6-24) -> (no net)
- U1 pad 6-25: Net-(U1-Pad6-25) -> (no net)
- U1 pad 6-26: Net-(U1-Pad6-26) -> (no net)
- U1 pad 6-27: Net-(U1-Pad6-27) -> (no net)
- U1 pad 6-28: Net-(U1-Pad6-28) -> (no net)
- U1 pad 6-29: Net-(U1-Pad6-29) -> (no net)
- U1 pad 6-30: Net-(U1-Pad6-30) -> (no net)
- U1 pad 6-31: Net-(U1-Pad6-31) -> (no net)
- U1 pad 6-32: Net-(U1-Pad6-32) -> (no net)
- U1 pad 6-33: Net-(U1-Pad6-33) -> (no net)
- U1 pad 6-34: Net-(U1-Pad6-34) -> (no net)
- U1 pad 6-35: Net-(U1-Pad6-35) -> (no net)
- U1 pad 6-36: Net-(U1-Pad6-36) -> (no net)
- U1 pad 6-37: Net-(U1-Pad6-37) -> (no net)
- U1 pad 6-38: Net-(U1-Pad6-38) -> (no net)
- U1 pad 6-39: Net-(U1-Pad6-39) -> (no net)
- U1 pad 6-40: Net-(U1-Pad6-40) -> (no net)
- U1 pad 6-5: Net-(U1-Pad6-5) -> (no net)
- U1 pad 6-6: Net-(U1-Pad6-6) -> (no net)
- U1 pad 6-7: Net-(U1-Pad6-7) -> (no net)
- U1 pad 6-8: Net-(U1-Pad6-8) -> (no net)
- U1 pad 6-9: Net-(U1-Pad6-9) -> (no net)
- U2 pad 5: Net-(U2-Pad5) -> (no net)
- U3 pad 10: Net-(P7-Pad2) -> Net-(P7-Pad3)
- U4 pad 4: Net-(R11-Pad2) -> PWR_LED
Routing:
- net GND: track 948.5 -> 0.00 mm, vias 14 -> 0
- net +5V: track 469.8 -> 0.00 mm, vias 6 -> 0
- net +3V3: track 303.6 -> 0.00 mm, vias 7 -> 0
- net PWR_LED: track 215.6 -> 0.00 mm, vias 3 -> 0
- net +6V: track 202.7 -> 0.00 mm, vias 5 -> 0
- net UART7_RX: track 150.4 -> 0.00 mm, vias 2 -> 0
- net TWI1_SDA: track 133.6 -> 0.00 mm, vias 2 -> 0
- net SAT_LED: track 127.1 -> 0.00 mm, vias 2 -> 0
- net GPS_LED: track 121.4 -> 0.00 mm, vias 2 -> 0
- net TWI1_SCK: track 120.6 -> 0.00 mm, vias 2 -> 0
- net UART3_RX: track 100.5 -> 0.00 mm, vias 1 -> 0
- net PG8: track 94.6 -> 0.00 mm, vias 1 -> 0
- net PG10: track 89.8 -> 0.00 mm, vias 1 -> 0
- net PG9: track 88.5 -> 0.00 mm, vias 1 -> 0
- net PG6: track 87.5 -> 0.00 mm, vias 1 -> 0
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
Commit message: thuraya datasheets
Parts:
- C59: moved to B.Cu
- moved R61 130.8 mm to (193.2, 35.6), turned to 90 degrees
- moved R47 121.5 mm to (174.1, 37.9), turned to 270 degrees
- moved C59 111.9 mm to (182.4, 51.4), turned to 270 degrees
- moved C53 98.8 mm to (169.7, 60.4), turned to 270 degrees
- moved R57 96.9 mm to (180.1, 66.9)
- moved R44 96.6 mm to (175.9, 65.2), turned to 180 degrees
- moved R43 95.1 mm to (175.9, 66.9), turned to 180 degrees
- moved C64 93.6 mm to (157.7, 62.3)
- moved L12 93.4 mm to (176.2, 68.9)
- moved C62 92.0 mm to (157.7, 63.9)
- moved R60 91.5 mm to (175.9, 70.8)
- moved C51 90.4 mm to (157.7, 65.6)
- moved R62 90.0 mm to (175.8, 72.5)
- moved C50 88.9 mm to (157.7, 67.1)
- moved R59 88.1 mm to (176.5, 75.0), turned to 180 degrees
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Connections:
- R1 pad 2: +5V -> +5VD
Routing:
- net GND: track 0.00 -> 1025.5 mm, vias 0 -> 56
- net +5V: track 0.00 -> 370.5 mm, vias 0 -> 3
- net +3V3: track 0.00 -> 223.6 mm
- net PWR_LED: track 0.00 -> 218.7 mm
- net SAT_LED: track 0.00 -> 208.8 mm
- net +6V: track 0.00 -> 207.6 mm, vias 0 -> 2
- net Net-(R10-Pad2): track 0.00 -> 150.0 mm, vias 0 -> 2
- net Net-(R11-Pad2): track 0.00 -> 131.5 mm, vias 0 -> 2
- net +5VD: track 0.00 -> 129.4 mm, vias 0 -> 2
- net GPS_LED: track 0.00 -> 121.6 mm, vias 0 -> 2
- net UART3_RX: track 0.00 -> 103.2 mm, vias 0 -> 1
- net PG9: track 0.00 -> 95.1 mm, vias 0 -> 1
- net PG10: track 0.00 -> 94.9 mm, vias 0 -> 1
- net PG6: track 0.00 -> 93.5 mm, vias 0 -> 1
- net PG8: track 0.00 -> 92.5 mm, vias 0 -> 1
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Other:
- board size 160.3 x 110.1 mm -> 174.4 x 110.1 mm
